Commit message: add ft ros2 control

File: tiago_pro_description/ros2_control/ros2_control.urdf.xacro (robot description, xacro)
@@ -84,10 +84,4 @@
         <xacro:ros2_control_arm name="arm_teleop_left_7" reduction="101.0" offset_value="${arm_left_7_joint_offset}" use_sea_transmission="${torque_estimation}" />
         </xacro:if>
-      <!-- <xacro:if value="${end_effector_right == 'pal-pro-gripper'}">
-        <xacro:ros2_control_pal_pro_gripper name="gripper_teleop_right" reduction="1.0" />
-      </xacro:if> -->
-      <!-- <xacro:if value="${end_effector_left == 'pal-pro-gripper'}">
-        <xacro:ros2_control_pal_pro_gripper name="gripper_teleop_left" reduction="1.0" />
-      </xacro:if> -->
     </xacro:if>
   </xacro:macro>
@@ -104,4 +98,6 @@
     <xacro:arg name="ft_sensor_left" default="no-ft-sensor"/>
     <xacro:arg name="ft_sensor_right" default="no-ft-sensor"/>
+    <xacro:arg name="ft_sensor_teleop_left" default="no-ft-sensor"/>
+    <xacro:arg name="ft_sensor_teleop_right" default="no-ft-sensor"/>
     <xacro:arg name="calibration_offset_dir" default="$(find tiago_pro_description)/urdf/calibration" />
     <!-- TODO-->
@@ -112,4 +108,6 @@
     <xacro:property name="has_ft_sensor_left" value="${ft_sensor_left != 'no-ft-sensor'}" />
     <xacro:property name="has_ft_sensor_right" value="${ft_sensor_right != 'no-ft-sensor'}" />
+    <xacro:property name="has_teleop_ft_sensor_left" value="${ft_sensor_teleop_left != 'no-ft-sensor'}" />
+    <xacro:property name="has_teleop_ft_sensor_right" value="${ft_sensor_teleop_right != 'no-ft-sensor'}" />
     <xacro:property name="has_arm_left" value="${arm_type_left != 'no-arm'}" />
     <xacro:property name="has_arm_right" value="${arm_type_right != 'no-arm'}" />

Commit message: offset

File: tiago_pro_description/ros2_control/ros2_control.urdf.xacro (robot description, xacro)
@@ -66,5 +66,5 @@
     </xacro:if>
   </xacro:macro>
-  <xacro:macro name="ros2_control_head">
+  <xacro:macro name="ros2_control_heads">
     <!-- head -->
     <xacro:ros2_control_head_joint name="head_1" offset_value="${head_1_joint_offset}" />
@@ -118,5 +118,5 @@
         <xacro:ros2_control_torso name="torso_lift" reduction="1.0" />
         <!-- head -->
-        <xacro:ros2_control_head />
+        <xacro:ros2_control_heads />
         <!-- arms -->
         <xacro:ros2_control_arms/>
@@ -148,5 +148,5 @@
         </hardware>
         <!-- head -->
-        <xacro:ros2_control_head />
+        <xacro:ros2_control_heads />
       </ros2_control>
       <!-- Ethercat system -->

Commit message: head_offset

File: tiago_pro_description/ros2_control/ros2_control.urdf.xacro (robot description, xacro)
@@ -66,5 +66,5 @@
     </xacro:if>
   </xacro:macro>
-  <xacro:macro name="ros2_control_heads">
+  <xacro:macro name="ros2_control_head">
     <!-- head -->
     <xacro:ros2_control_head_joint name="head_1" offset_value="${head_1_joint_offset}" reduction="1.0"/>
@@ -118,5 +118,5 @@
         <xacro:ros2_control_torso name="torso_lift" reduction="1.0" />
         <!-- head -->
-        <xacro:ros2_control_heads />
+        <xacro:ros2_control_head />
         <!-- arms -->
         <xacro:ros2_control_arms/>
@@ -148,5 +148,5 @@
         </hardware>
         <!-- head -->
-        <xacro:ros2_control_heads />
+        <xacro:ros2_control_head />
       </ros2_control>
       <!-- Ethercat system -->

Commit message: changes for head_offset

File: tiago_pro_description/ros2_control/ros2_control.urdf.xacro (robot description, xacro)
@@ -65,9 +65,4 @@
       </xacro:if>
     </xacro:if>
-  </xacro:macro>
-  <xacro:macro name="ros2_control_head">
-    <!-- head -->
-    <xacro:ros2_control_head_joint name="head_1" offset_value="${head_1_joint_offset}" reduction="1.0"/>
-    <xacro:ros2_control_head_joint name="head_2" offset_value="${head_2_joint_offset}" reduction="1.0"/>
   </xacro:macro>
   <xacro:macro name="tiago_pro_ros2_control" params="use_sim_time:=^|false">

Commit message: changes for head_offset

File: tiago_pro_description/ros2_control/ros2_control.urdf.xacro (robot description, xacro)
@@ -66,4 +66,9 @@
     </xacro:if>
   </xacro:macro>
+  <xacro:macro name="ros2_control_head_offset">
+    <!-- head -->
+    <xacro:ros2_control_head_joint name="head_1" reduction="1.0" offset_value="${head_1_joint_offset}" />
+    <xacro:ros2_control_head_joint name="head_2" reduction="1.0" offset_value="${head_2_joint_offset}" />
+  </xacro:macro>
   <xacro:macro name="tiago_pro_ros2_control" params="use_sim_time:=^|false">
     <xacro:arg name="arm_type_left" default="tiago-pro"/>
@@ -113,5 +118,5 @@
         <xacro:ros2_control_torso name="torso_lift" reduction="1.0" />
         <!-- head -->
-        <xacro:ros2_control_head />
+        <xacro:ros2_control_head_offset />
         <!-- arms -->
         <xacro:ros2_control_arms/>
@@ -143,5 +148,5 @@
         </hardware>
         <!-- head -->
-        <xacro:ros2_control_head />
+        <xacro:ros2_control_head_offset />
       </ros2_control>
       <!-- Ethercat system -->
