Commit message: fix urdf

File: tiago_pro_description/robots/tiago_pro.urdf.xacro (robot description, xacro)
@@ -20,4 +20,6 @@
   <!-- tiago-pro, no-arm -->
   <xacro:arg name="arm_type_right" default="tiago-pro" />
+  <xacro:arg name="arm_type_teleop_right" default="tiago-pro" />
+  <xacro:arg name="arm_type_teleop_left" default="tiago-pro" />
   <!-- straight-wrist, spherical-wrist -->
   <xacro:arg name="wrist_model_left" default="spherical-wrist" />
@@ -65,4 +67,6 @@
   <xacro:property name="arm_type_left" value="$(arg arm_type_left)" />
   <xacro:property name="arm_type_right" value="$(arg arm_type_right)" />
+  <xacro:property name="arm_type_teleop_left" value="$(arg arm_type_teleop_left)" />
+  <xacro:property name="arm_type_teleop_right" value="$(arg arm_type_teleop_right)" />
   <xacro:property name="tool_changer_left" value="$(arg tool_changer_left)" />
   <xacro:property name="tool_changer_right" value="$(arg tool_changer_right)" />
@@ -82,4 +86,6 @@
   <xacro:property name="end_effector_left_name" value="gripper_left" />
   <xacro:property name="has_arm_right" value="${arm_type_right not in ['no-arm']}"/>
+  <xacro:property name="has_teleop_arm_right" value="${arm_type_teleop_right not in ['no-arm']}"/>
+  <xacro:property name="has_teleop_arm_left" value="${arm_type_teleop_left not in ['no-arm']}"/>
   <xacro:property name="has_ft_sensor_right" value="${ft_sensor_right not in ['no-ft-sensor']}"/>
   <xacro:property name="has_end_effector_right" value="${end_effector_right not in ['no-end-effector']}" />
@@ -92,4 +98,10 @@
   <xacro:if value="${arm_type_right not in ['tiago-pro-prototype', 'tiago-pro', 'tiago-pro-s', 'no-arm']}">
     <xacro:wrong_arm_type_right />
+  </xacro:if>
+  <xacro:if value="${arm_type_teleop_left not in ['tiago-pro-prototype', 'tiago-pro', 'tiago-pro-s', 'no-arm']}">
+    <xacro:wrong_arm_type_teleop_left />
+  </xacro:if>
+  <xacro:if value="${arm_type_teleop_right not in ['tiago-pro-prototype', 'tiago-pro', 'tiago-pro-s', 'no-arm']}">
+    <xacro:wrong_arm_type_teleop_right />
   </xacro:if>
   <xacro:if value="${end_effector_left not in ['pal-pro-gripper', 'custom', 'no-end-effector', 'allegro-hand']}">
@@ -206,16 +218,16 @@
   <!-- Teleop arms without FT -->
   <xacro:if value="${has_teleop_arms}">
-    <xacro:pal_sea_arm name="arm_teleop_right" parent="torso_lift_link" arm_type="${arm_type_right}" wrist_model="${wrist_model_right}" tool_changer="${tool_changer_right}" reflect="1" joint_reflect="1" arm_1_offset="${arm_right_1_joint_offset}" arm_2_offset="${arm_right_2_joint_offset}" arm_3_offset="${arm_right_3_joint_offset}" arm_4_offset="${arm_right_4_joint_offset}" arm_5_offset="${arm_right_5_joint_offset}" arm_6_offset="${arm_right_6_joint_offset}" arm_7_offset="${arm_right_7_joint_offset}">
+    <xacro:pal_sea_arm name="arm_teleop_right" parent="torso_lift_link" arm_type="${arm_type_teleop_right}" wrist_model="${wrist_model_right}" tool_changer="${tool_changer_right}" reflect="1" joint_reflect="1" arm_1_offset="${arm_right_1_joint_offset}" arm_2_offset="${arm_right_2_joint_offset}" arm_3_offset="${arm_right_3_joint_offset}" arm_4_offset="${arm_right_4_joint_offset}" arm_5_offset="${arm_right_5_joint_offset}" arm_6_offset="${arm_right_6_joint_offset}" arm_7_offset="${arm_right_7_joint_offset}">
       <origin xyz="$(arg arm_x) ${-12*$(arg arm_y)} $(arg arm_z)" rpy="$(arg arm_roll) ${-11.0*$(arg arm_pitch)} ${-3.14159 -$(arg arm_yaw)}"/>
     </xacro:pal_sea_arm>
-    <xacro:pal_sea_arm name="arm_teleop_left" parent="torso_lift_link" arm_type="${arm_type_left}" wrist_model="${wrist_model_left}" tool_changer="${tool_changer_left}" reflect="1" joint_reflect="-1" arm_1_offset="${arm_left_1_joint_offset}" arm_2_offset="${arm_left_2_joint_offset}" arm_3_offset="${arm_left_3_joint_offset}" arm_4_offset="${arm_left_4_joint_offset}" arm_5_offset="${arm_left_5_joint_offset}" arm_6_offset="${arm_left_6_joint_offset}" arm_7_offset="${arm_left_7_joint_offset}">
+    <xacro:pal_sea_arm name="arm_teleop_left" parent="torso_lift_link" arm_type="${arm_type_teleop_left}" wrist_model="${wrist_model_left}" tool_changer="${tool_changer_left}" reflect="1" joint_reflect="-1" arm_1_offset="${arm_left_1_joint_offset}" arm_2_offset="${arm_left_2_joint_offset}" arm_3_offset="${arm_left_3_joint_offset}" arm_4_offset="${arm_left_4_joint_offset}" arm_5_offset="${arm_left_5_joint_offset}" arm_6_offset="${arm_left_6_joint_offset}" arm_7_offset="${arm_left_7_joint_offset}">
       <origin xyz="$(arg arm_x) ${-10.0*$(arg arm_y)} $(arg arm_z)" rpy="$(arg arm_roll) $(arg arm_pitch) $(arg arm_yaw)"/>
     </xacro:pal_sea_arm>
-    <xacro:if value="${has_end_effector_left}">
+    <!-- <xacro:if value="${has_end_effector_left}">
       <xacro:pal_sea_arm_end_effector name="gripper_teleop_left" parent="arm_teleop_left_tool_link" type="${end_effector_left}" tool_changer="${tool_changer_left}" reflect="-1"/>
     </xacro:if>
     <xacro:if value="${has_end_effector_right}">
       <xacro:pal_sea_arm_end_effector name="gripper_teleop_right" parent="arm_teleop_right_tool_link" type="${end_effector_right}" tool_changer="${tool_changer_right}" reflect="1"/>
-    </xacro:if>
+    </xacro:if> -->
   </xacro:if>
   <!-- ROS 2 Control -->

File: tiago_pro_description/ros2_control/ros2_control.urdf.xacro (robot description, xacro)
@@ -65,4 +65,27 @@
       </xacro:if>
     </xacro:if>
+    <xacro:if value="${has_teleop_arms}">
+      <xacro:ros2_control_arm name="arm_teleop_right_1" reduction="121.0" offset_value="${arm_right_1_joint_offset}" use_sea_transmission="${torque_estimation}" />
+      <xacro:ros2_control_arm name="arm_teleop_right_2" reduction="121.0" offset_value="${arm_right_2_joint_offset}" use_sea_transmission="${torque_estimation}" />
+      <xacro:ros2_control_arm name="arm_teleop_right_3" reduction="101.0" offset_value="${arm_right_3_joint_offset}" use_sea_transmission="${torque_estimation}" />
+      <xacro:ros2_control_arm name="arm_teleop_right_4" reduction="101.0" offset_value="${arm_right_4_joint_offset}" use_sea_transmission="${torque_estimation}" />
+      <xacro:ros2_control_arm name="arm_teleop_right_5" reduction="101.0" offset_value="${arm_right_5_joint_offset}" use_sea_transmission="${torque_estimation}" />
+      <xacro:ros2_control_arm name="arm_teleop_right_6" reduction="101.0" offset_value="${arm_right_6_joint_offset}" use_sea_transmission="${torque_estimation}" />
+      <xacro:ros2_control_arm name="arm_teleop_right_7" reduction="101.0" offset_value="${arm_right_7_joint_offset}" use_sea_transmission="${torque_estimation}" />
+      <xacro:ros2_control_arm name="arm_teleop_left_1" reduction="121.0" offset_value="${arm_left_1_joint_offset}" use_sea_transmission="${torque_estimation}" />
+      <xacro:ros2_control_arm name="arm_teleop_left_2" reduction="121.0" offset_value="${arm_left_2_joint_offset}" use_sea_transmission="${torque_estimation}" />
+      <xacro:ros2_control_arm name="arm_teleop_left_3" reduction="101.0" offset_value="${arm_left_3_joint_offset}" use_sea_transmission="${torque_estimation}" />
+      <xacro:ros2_control_arm name="arm_teleop_left_4" reduction="101.0" offset_value="${arm_left_4_joint_offset}" use_sea_transmission="${torque_estimation}" />
+      <xacro:ros2_control_arm name="arm_teleop_left_5" reduction="101.0" offset_value="${arm_left_5_joint_offset}" use_sea_transmission="${torque_estimation}" />
+      <xacro:ros2_control_arm name="arm_teleop_left_6" reduction="101.0" offset_value="${arm_left_6_joint_offset}" use_sea_transmission="${torque_estimation}" />
+      <xacro:ros2_control_arm name="arm_teleop_left_7" reduction="101.0" offset_value="${arm_left_7_joint_offset}" use_sea_transmission="${torque_estimation}" />
+      <xacro:if value="${end_effector_right == 'pal-pro-gripper'}">
+        <!-- pal-pro-gripper -->
+        <xacro:ros2_control_pal_pro_gripper name="gripper_teleop_right" reduction="1.0" />
+      </xacro:if>
+      <xacro:if value="${end_effector_left == 'pal-pro-gripper'}">
+        <xacro:ros2_control_pal_pro_gripper name="gripper_teleop_left" reduction="1.0" />
+      </xacro:if>
+    </xacro:if>
   </xacro:macro>
   <xacro:macro name="ros2_control_head_offset">
@@ -71,5 +94,5 @@
     <xacro:ros2_control_head_joint name="head_2" reduction="1.0" offset_value="${head_2_joint_offset}" />
   </xacro:macro>
-  <xacro:macro name="tiago_pro_ros2_control" params="use_sim_time:=^|false">
+  <xacro:macro name="tiago_pro_ros2_control" params="use_sim_time:=^|false has_teleop_arms:=^|false">
     <xacro:arg name="arm_type_left" default="tiago-pro"/>
     <xacro:arg name="arm_type_right" default="tiago-pro"/>

Commit message: fix FT sensors after rebase

File: tiago_pro_description/robots/tiago_pro.urdf.xacro (robot description, xacro)
@@ -30,4 +30,8 @@
   <!-- False, True -->
   <xacro:arg name="tool_changer_left" default="True" />
+    <!-- False, True -->
+  <xacro:arg name="tool_changer_teleop_right" default="True" />
+  <!-- False, True -->
+  <xacro:arg name="tool_changer_teleop_left" default="True" />
   <!-- pal-pro-gripper custom-->
   <xacro:arg name="end_effector_left" default="pal-pro-gripper" />
@@ -38,4 +42,8 @@
   <!-- no-ft-sensor, rokubi -->
   <xacro:arg name="ft_sensor_right" default="no-ft-sensor" />
+  <!-- no-ft-sensor, rokubi -->
+  <xacro:arg name="ft_sensor_teleop_left" default="no-ft-sensor" />
+  <!-- no-ft-sensor, rokubi -->
+  <xacro:arg name="ft_sensor_teleop_right" default="no-ft-sensor" />
   <!-- realsense-d435 -->
   <xacro:arg name="camera_model" default="realsense-d435" />
@@ -71,4 +79,6 @@
   <xacro:property name="tool_changer_left" value="$(arg tool_changer_left)" />
   <xacro:property name="tool_changer_right" value="$(arg tool_changer_right)" />
+  <xacro:property name="tool_changer_teleop_left" value="$(arg tool_changer_teleop_left)" />
+  <xacro:property name="tool_changer_teleop_right" value="$(arg tool_changer_teleop_right)" />
   <xacro:property name="wrist_model_left" value="$(arg wrist_model_left)" />
   <xacro:property name="wrist_model_right" value="$(arg wrist_model_right)" />
@@ -77,4 +87,6 @@
   <xacro:property name="ft_sensor_left" value="$(arg ft_sensor_left)" />
   <xacro:property name="ft_sensor_right" value="$(arg ft_sensor_right)" />
+  <xacro:property name="ft_sensor_teleop_left" value="$(arg ft_sensor_teleop_left)" />
+  <xacro:property name="ft_sensor_teleop_right" value="$(arg ft_sensor_teleop_right)" />
   <xacro:property name="camera_model" value="$(arg camera_model)" />
   <xacro:property name="calibration_offset_dir" value="${arg calibration_offset_dir}"/>
@@ -89,6 +101,10 @@
   <xacro:property name="has_teleop_arm_left" value="${arm_type_teleop_left not in ['no-arm']}"/>
   <xacro:property name="has_ft_sensor_right" value="${ft_sensor_right not in ['no-ft-sensor']}"/>
+  <xacro:property name="has_teleop_ft_sensor_right" value="${ft_sensor_teleop_right not in ['no-ft-sensor']}"/>
+  <xacro:property name="has_teleop_ft_sensor_left" value="${ft_sensor_teleop_left not in ['no-ft-sensor']}"/>
   <xacro:property name="has_end_effector_right" value="${end_effector_right not in ['no-end-effector']}" />
   <xacro:property name="end_effector_right_link" value="${'wrist_right_ft_tool_link' if has_ft_sensor_right else 'arm_right_tool_link'}" />
+  <xacro:property name="end_effector_teleop_right_link" value="${'wrist_teleop_right_ft_tool_link' if has_teleop_ft_sensor_right else 'arm_teleop_right_tool_link'}" />
+  <xacro:property name="end_effector_teleop_left_link" value="${'wrist_teleop_left_ft_tool_link' if has_teleop_ft_sensor_left else 'arm_teleop_left_tool_link'}" />
   <xacro:property name="end_effector_right_name" value="gripper_right" />
   <!-- Properties check -->
@@ -116,4 +132,10 @@
   <xacro:if value="${ft_sensor_right not in ['no-ft-sensor', 'rokubi', 'ati']}">
     <xacro:wrong_ft_sensor_right />
+  </xacro:if>
+  <xacro:if value="${ft_sensor_teleop_left not in ['no-ft-sensor', 'rokubi', 'ati']}">
+    <xacro:wrong_ft_sensor_teleop_left />
+  </xacro:if>
+  <xacro:if value="${ft_sensor_teleop_right not in ['no-ft-sensor', 'rokubi', 'ati']}">
+    <xacro:wrong_ft_sensor_teleop_right />
   </xacro:if>
   <xacro:if value="${laser_model not in ['no-laser', 'sick-571']}">
@@ -169,5 +191,5 @@
   </xacro:if>
   <!-- Force Torque sensor -->
-  <xacro:if value="${has_ft_sensor_right or has_ft_sensor_left}">
+  <xacro:if value="${has_ft_sensor_right or has_ft_sensor_left or has_teleop_ft_sensor_right or has_teleop_ft_sensor_left}">
     <xacro:include filename="$(find pal_urdf_utils)/urdf/ft_sensors/ft_sensor.urdf.xacro" />
     <xacro:include filename="$(find pal_urdf_utils)/urdf/ft_sensors/ft_sensor.gazebo.xacro" />
@@ -218,16 +240,16 @@
   <!-- Teleop arms without FT -->
   <xacro:if value="${has_teleop_arms}">
-    <xacro:pal_sea_arm name="arm_teleop_right" parent="torso_lift_link" arm_type="${arm_type_teleop_right}" wrist_model="${wrist_model_right}" tool_changer="${tool_changer_right}" reflect="1" joint_reflect="1" arm_1_offset="${arm_right_1_joint_offset}" arm_2_offset="${arm_right_2_joint_offset}" arm_3_offset="${arm_right_3_joint_offset}" arm_4_offset="${arm_right_4_joint_offset}" arm_5_offset="${arm_right_5_joint_offset}" arm_6_offset="${arm_right_6_joint_offset}" arm_7_offset="${arm_right_7_joint_offset}">
+    <xacro:pal_sea_arm name="arm_teleop_right" parent="torso_lift_link" arm_type="${arm_type_teleop_right}" wrist_model="${wrist_model_right}" tool_changer="${tool_changer_teleop_right}" reflect="1" joint_reflect="1" arm_1_offset="${arm_right_1_joint_offset}" arm_2_offset="${arm_right_2_joint_offset}" arm_3_offset="${arm_right_3_joint_offset}" arm_4_offset="${arm_right_4_joint_offset}" arm_5_offset="${arm_right_5_joint_offset}" arm_6_offset="${arm_right_6_joint_offset}" arm_7_offset="${arm_right_7_joint_offset}">
       <origin xyz="$(arg arm_x) ${-12*$(arg arm_y)} $(arg arm_z)" rpy="$(arg arm_roll) ${-11.0*$(arg arm_pitch)} ${-3.14159 -$(arg arm_yaw)}"/>
     </xacro:pal_sea_arm>
-    <xacro:pal_sea_arm name="arm_teleop_left" parent="torso_lift_link" arm_type="${arm_type_teleop_left}" wrist_model="${wrist_model_left}" tool_changer="${tool_changer_left}" reflect="1" joint_reflect="-1" arm_1_offset="${arm_left_1_joint_offset}" arm_2_offset="${arm_left_2_joint_offset}" arm_3_offset="${arm_left_3_joint_offset}" arm_4_offset="${arm_left_4_joint_offset}" arm_5_offset="${arm_left_5_joint_offset}" arm_6_offset="${arm_left_6_joint_offset}" arm_7_offset="${arm_left_7_joint_offset}">
+    <xacro:pal_sea_arm name="arm_teleop_left" parent="torso_lift_link" arm_type="${arm_type_teleop_left}" wrist_model="${wrist_model_left}" tool_changer="${tool_changer_teleop_left}" reflect="1" joint_reflect="-1" arm_1_offset="${arm_left_1_joint_offset}" arm_2_offset="${arm_left_2_joint_offset}" arm_3_offset="${arm_left_3_joint_offset}" arm_4_offset="${arm_left_4_joint_offset}" arm_5_offset="${arm_left_5_joint_offset}" arm_6_offset="${arm_left_6_joint_offset}" arm_7_offset="${arm_left_7_joint_offset}">
       <origin xyz="$(arg arm_x) ${-10.0*$(arg arm_y)} $(arg arm_z)" rpy="$(arg arm_roll) $(arg arm_pitch) $(arg arm_yaw)"/>
     </xacro:pal_sea_arm>
-    <!-- <xacro:if value="${has_end_effector_left}">
-      <xacro:pal_sea_arm_end_effector name="gripper_teleop_left" parent="arm_teleop_left_tool_link" type="${end_effector_left}" tool_changer="${tool_changer_left}" reflect="-1"/>
-    </xacro:if>
-    <xacro:if value="${has_end_effector_right}">
-      <xacro:pal_sea_arm_end_effector name="gripper_teleop_right" parent="arm_teleop_right_tool_link" type="${end_effector_right}" tool_changer="${tool_changer_right}" reflect="1"/>
-    </xacro:if> -->
+    <xacro:if value="${has_teleop_ft_sensor_right}">
+      <xacro:ft_sensor type="${ft_sensor_teleop_right}" name="wrist_teleop_right" parent="arm_teleop_right_tool_link"/>
+    </xacro:if>
+    <xacro:if value="${has_teleop_ft_sensor_left}">
+      <xacro:ft_sensor type="${ft_sensor_teleop_left}" name="wrist_teleop_left" parent="arm_teleop_left_tool_link"/>
+    </xacro:if>
   </xacro:if>
   <!-- ROS 2 Control -->

File: tiago_pro_description/ros2_control/ros2_control.urdf.xacro (robot description, xacro)
@@ -84,4 +84,12 @@
         <xacro:ros2_control_arm name="arm_teleop_left_7" reduction="101.0" offset_value="${arm_left_7_joint_offset}" use_sea_transmission="${torque_estimation}" />
         </xacro:if>
+      <xacro:if value="${has_teleop_ft_sensor_right}">
+        <xacro:include filename="$(find pal_urdf_utils)/urdf/ft_sensors/ftsensor.ros2_control.xacro"/>
+        <xacro:ros2_control_force_torque_sensor name="wrist_teleop_right_ft_sensor"/>
+      </xacro:if>
+      <xacro:if value="${has_teleop_ft_sensor_left}">
+        <xacro:include filename="$(find pal_urdf_utils)/urdf/ft_sensors/ftsensor.ros2_control.xacro"/>
+        <xacro:ros2_control_force_torque_sensor name="wrist_teleop_left_ft_sensor"/>
+      </xacro:if>
     </xacro:if>
   </xacro:macro>

Commit message: Add urdf calibration args for the arm

File: tiago_pro_description/robots/tiago_pro.urdf.xacro (robot description, xacro)
@@ -44,5 +44,5 @@
   <xacro:arg name="is_multiple" default="false"/>
   <xacro:arg name="namespace" default=""/>
-  <xacro:arg name="description_calibration_dir" default="$(find tiago_pro_description)/urdf"/>
+  <xacro:arg name="arm_calibration_dir" default="$(find tiago_pro_description)/urdf/calibration"/>
   <xacro:arg name="extrinsic_calibration_dir" default="$(find tiago_pro_description)/urdf"/>
   <xacro:arg name="arm_x" default="0.08976" />
@@ -69,5 +69,5 @@
   <xacro:property name="ft_sensor_right" value="$(arg ft_sensor_right)" />
   <xacro:property name="camera_model" value="$(arg camera_model)" />
-  <xacro:property name="description_calibration_dir" value="${arg description_calibration_dir}"/>
+  <xacro:property name="arm_calibration_dir" value="${arg arm_calibration_dir}"/>
   <xacro:property name="is_public_sim" value="$(arg is_public_sim)" />
   <xacro:property name="has_arm_left" value="${arm_type_left not in ['no-arm']}"/>
@@ -142,5 +142,5 @@
   <xacro:include filename="$(find tiago_pro_description)/urdf/torso/torso.urdf.xacro" />
   <!-- Calibration constants -->
-  <xacro:include filename="$(arg description_calibration_dir)/calibration_constants.urdf.xacro" />
+  <xacro:include filename="$(arg arm_calibration_dir)/arm_calibration.urdf.xacro" />
   <!-- Arm -->
   <xacro:if value="${has_arm_right or has_arm_left}">

File: tiago_pro_description/ros2_control/ros2_control.urdf.xacro (robot description, xacro)
@@ -73,5 +73,5 @@
     <xacro:arg name="ft_sensor_left" default="no-ft-sensor"/>
     <xacro:arg name="ft_sensor_right" default="no-ft-sensor"/>
-    <xacro:arg name="description_calibration_dir" default="$(find tiago_pro_description)/urdf/calibration" />
+    <xacro:arg name="arm_calibration_dir" default="$(find tiago_pro_description)/urdf/calibration" />
     <!-- TODO-->
     <xacro:property name="arm_type_left" value="$(arg arm_type_left)" />
@@ -95,5 +95,5 @@
     </xacro:if>
     <!-- calibration offsets -->
-    <xacro:include filename="$(arg description_calibration_dir)/calibration_constants.urdf.xacro" />
+    <xacro:include filename="$(arg arm_calibration_dir)/arm_calibration.urdf.xacro" />
     <!-- Simulation -->
     <xacro:if value="$(arg use_sim_time)">

File: tiago_pro_description/urdf/calibration/arm_calibration.urdf.xacro (robot description, xacro)
@@ -6,13 +6,4 @@
 <robot xmlns:xacro="http://ros.org/wiki/xacro">
 	<!--Constant parameters-->
-	<xacro:property name="camera_position_x" value="0.0908" />
-	<xacro:property name="camera_position_y" value="0.08" />
-	<xacro:property name="camera_position_z" value="0.0" />
-	<xacro:property name="camera_orientation_r" value="${-90 * deg_to_rad}" />
-	<xacro:property name="camera_orientation_p" value="0.0" />
-	<xacro:property name="camera_orientation_y" value="0.0" />
-	<xacro:property name="head_2_joint_offset" value="0" />
-	<xacro:property name="head_1_joint_offset" value="0" />
-	<xacro:property name="torso_lift_joint_offset" value="0" />
 	<xacro:property name="arm_left_1_joint_offset" value="0.0" />
 	<xacro:property name="arm_left_2_joint_offset" value="0.0" />

Commit message: adding head calibration offset

File: tiago_pro_description/robots/tiago_pro.urdf.xacro (robot description, xacro)
@@ -144,5 +144,5 @@
   <xacro:include filename="$(find tiago_pro_description)/urdf/torso/torso.urdf.xacro" />
   <!-- Calibration constants -->
-  <xacro:include filename="$(arg arm_calibration_dir)/arm_calibration.urdf.xacro" />
+  <xacro:include filename="$(arg arm_calibration_dir)/calibration_offset.urdf.xacro" />
   <!-- Arm -->
   <xacro:if value="${has_arm_right or has_arm_left}">

File: tiago_pro_description/ros2_control/ros2_control.urdf.xacro (robot description, xacro)
@@ -66,4 +66,9 @@
     </xacro:if>
   </xacro:macro>
+  <xacro:macro name="ros2_control_head">
+    <!-- head -->
+    <xacro:ros2_control_head_joint name="head_1" offset_value="${head_1_joint_offset}" />
+    <xacro:ros2_control_head_joint name="head_2" offset_value="${head_2_joint_offset}" />
+  </xacro:macro>
   <xacro:macro name="tiago_pro_ros2_control" params="use_sim_time:=^|false">
     <xacro:arg name="arm_type_left" default="tiago-pro"/>
@@ -95,5 +100,5 @@
     </xacro:if>
     <!-- calibration offsets -->
-    <xacro:include filename="$(arg arm_calibration_dir)/arm_calibration.urdf.xacro" />
+    <xacro:include filename="$(arg arm_calibration_dir)/calibration_offset.urdf.xacro" />
     <!-- Simulation -->
     <xacro:if value="$(arg use_sim_time)">

File: tiago_pro_description/urdf/calibration/calibration_offset.urdf.xacro (robot description, xacro)
@@ -20,3 +20,5 @@
   	<xacro:property name="arm_right_6_joint_offset" value="0.0" />
   	<xacro:property name="arm_right_7_joint_offset" value="0.0" />
-</robot>
+	<xacro:property name="head_1_joint_offset" value="0.0" />
+  	<xacro:property name="head_2_joint_offset" value="0.0" />
+</robot>ll
