Commit message: add teleop arms in the urdf

File: tiago_pro_description/robots/tiago_pro.urdf.xacro (robot description, xacro)
@@ -41,4 +41,6 @@
   <xacro:arg name="torque_estimation" default="False" />
   <xacro:arg name="gazebo_version" default="classic"/>
+  <!-- False, True -->
+  <xacro:arg name="has_teleop_arms" default="False" />
   <xacro:arg name="use_sim_time" default="false"/>
   <xacro:arg name="is_public_sim" default="false"/>
@@ -56,4 +58,5 @@
   <xacro:property name="torque_estimation" value="$(arg torque_estimation)" />
   <xacro:property name="gazebo_version" value="$(arg gazebo_version)" />
+  <xacro:property name="has_teleop_arms" value="$(arg has_teleop_arms)" />
   <xacro:property name="use_sim_time" value="$(arg use_sim_time)" />
   <xacro:property name="is_multiple" value="$(arg is_multiple)" />
@@ -201,5 +204,20 @@
     </xacro:if>
   </xacro:if>
+  <!-- Teleop arms without FT -->
+  <xacro:if value="${has_teleop_arms}">
+    <xacro:pal_sea_arm name="arm_teleop_right" parent="torso_lift_link" arm_type="${arm_type_right}" wrist_model="${wrist_model_right}" tool_changer="${tool_changer_right}" reflect="1" joint_reflect="1" arm_1_offset="${arm_right_1_joint_offset}" arm_2_offset="${arm_right_2_joint_offset}" arm_3_offset="${arm_right_3_joint_offset}" arm_4_offset="${arm_right_4_joint_offset}" arm_5_offset="${arm_right_5_joint_offset}" arm_6_offset="${arm_right_6_joint_offset}" arm_7_offset="${arm_right_7_joint_offset}">
+      <origin xyz="$(arg arm_x) ${-12*$(arg arm_y)} $(arg arm_z)" rpy="$(arg arm_roll) ${-11.0*$(arg arm_pitch)} ${-3.14159 -$(arg arm_yaw)}"/>
+    </xacro:pal_sea_arm>
+    <xacro:pal_sea_arm name="arm_teleop_left" parent="torso_lift_link" arm_type="${arm_type_left}" wrist_model="${wrist_model_left}" tool_changer="${tool_changer_left}" reflect="1" joint_reflect="1" arm_1_offset="${arm_left_1_joint_offset}" arm_2_offset="${arm_left_2_joint_offset}" arm_3_offset="${arm_left_3_joint_offset}" arm_4_offset="${arm_left_4_joint_offset}" arm_5_offset="${arm_left_5_joint_offset}" arm_6_offset="${arm_left_6_joint_offset}" arm_7_offset="${arm_left_7_joint_offset}">
+      <origin xyz="$(arg arm_x) ${-10.0*$(arg arm_y)} $(arg arm_z)" rpy="$(arg arm_roll) $(arg arm_pitch) $(arg arm_yaw)"/>
+    </xacro:pal_sea_arm>
+    <xacro:if value="${has_end_effector_left}">
+      <xacro:pal_sea_arm_end_effector name="gripper_teleop_left" parent="arm_teleop_left_tool_link" type="${end_effector_left}" tool_changer="${tool_changer_left}" reflect="-1"/>
+    </xacro:if>
+    <xacro:if value="${has_end_effector_right}">
+      <xacro:pal_sea_arm_end_effector name="gripper_teleop_right" parent="arm_teleop_right_tool_link" type="${end_effector_right}" tool_changer="${tool_changer_right}" reflect="1"/>
+    </xacro:if>
+  </xacro:if>
   <!-- ROS 2 Control -->
-  <xacro:tiago_pro_ros2_control use_sim_time="$(arg use_sim_time)" />
+  <xacro:tiago_pro_ros2_control use_sim_time="$(arg use_sim_time)" has_teleop_arms="${has_teleop_arms}"/>
 </robot>

Commit message: rename calibration directory

File: tiago_pro_description/robots/tiago_pro.urdf.xacro (robot description, xacro)
@@ -45,5 +45,5 @@
   <xacro:arg name="is_multiple" default="false"/>
   <xacro:arg name="namespace" default=""/>
-  <xacro:arg name="arm_calibration_dir" default="$(find tiago_pro_description)/urdf/calibration"/>
+  <xacro:arg name="calibration_offset_dir" default="$(find tiago_pro_description)/urdf/calibration"/>
   <xacro:arg name="extrinsic_calibration_dir" default="$(find tiago_pro_description)/urdf"/>
   <xacro:arg name="arm_x" default="0.08976" />
@@ -71,5 +71,5 @@
   <xacro:property name="ft_sensor_right" value="$(arg ft_sensor_right)" />
   <xacro:property name="camera_model" value="$(arg camera_model)" />
-  <xacro:property name="arm_calibration_dir" value="${arg arm_calibration_dir}"/>
+  <xacro:property name="calibration_offset_dir" value="${arg calibration_offset_dir}"/>
   <xacro:property name="is_public_sim" value="$(arg is_public_sim)" />
   <xacro:property name="has_arm_left" value="${arm_type_left not in ['no-arm']}"/>
@@ -144,5 +144,5 @@
   <xacro:include filename="$(find tiago_pro_description)/urdf/torso/torso.urdf.xacro" />
   <!-- Calibration constants -->
-  <xacro:include filename="$(arg arm_calibration_dir)/calibration_offset.urdf.xacro" />
+  <xacro:include filename="$(arg calibration_offset_dir)/calibration_offset.urdf.xacro" />
   <!-- Arm -->
   <xacro:if value="${has_arm_right or has_arm_left}">

File: tiago_pro_description/ros2_control/ros2_control.urdf.xacro (robot description, xacro)
@@ -78,5 +78,5 @@
     <xacro:arg name="ft_sensor_left" default="no-ft-sensor"/>
     <xacro:arg name="ft_sensor_right" default="no-ft-sensor"/>
-    <xacro:arg name="arm_calibration_dir" default="$(find tiago_pro_description)/urdf/calibration" />
+    <xacro:arg name="calibration_offset_dir" default="$(find tiago_pro_description)/urdf/calibration" />
     <!-- TODO-->
     <xacro:property name="arm_type_left" value="$(arg arm_type_left)" />
@@ -100,5 +100,5 @@
     </xacro:if>
     <!-- calibration offsets -->
-    <xacro:include filename="$(arg arm_calibration_dir)/calibration_offset.urdf.xacro" />
+    <xacro:include filename="$(arg calibration_offset_dir)/calibration_offset.urdf.xacro" />
     <!-- Simulation -->
     <xacro:if value="$(arg use_sim_time)">

Commit message: Add new limits values

File: tiago_pro_description/robots/tiago_pro.urdf.xacro (robot description, xacro)
@@ -54,4 +54,6 @@
   <!-- realsense-d435 -->
   <xacro:arg name="camera_model" default="realsense-d435" />
+  <!-- limits v2 -->
+  <xacro:arg name="limits_v2" default="False" />
   <!-- False, True -->
   <xacro:arg name="torque_estimation" default="False" />
@@ -119,4 +121,5 @@
   <xacro:property name="end_effector_teleop_left_link" value="${'wrist_teleop_left_ft_tool_link' if has_teleop_ft_sensor_left else 'arm_teleop_left_tool_link'}" />
   <xacro:property name="end_effector_right_name" value="gripper_right" />
+  <xacro:property name="limits_v2" value="$(arg limits_v2)" />
   <xacro:property name="has_end_effector_teleop_left" value="${end_effector_teleop_left not in ['no-end-effector']}" />
   <xacro:property name="has_end_effector_teleop_right" value="${end_effector_teleop_right not in ['no-end-effector']}" />
@@ -254,5 +257,5 @@
   <xacro:if value="${has_arm_left}">
     <!-- Arm -->
-    <xacro:pal_sea_arm name="arm_left" parent="torso_lift_link" arm_type="${arm_type_left}" wrist_model="${wrist_model_left}" tool_changer="${tool_changer_left}" reflect="1" joint_reflect="-1" arm_1_offset="${arm_left_1_joint_offset}" arm_2_offset="${arm_left_2_joint_offset}" arm_3_offset="${arm_left_3_joint_offset}" arm_4_offset="${arm_left_4_joint_offset}" arm_5_offset="${arm_left_5_joint_offset}" arm_6_offset="${arm_left_6_joint_offset}" arm_7_offset="${arm_left_7_joint_offset}">
+    <xacro:pal_sea_arm name="arm_left" parent="torso_lift_link" arm_type="${arm_type_left}" wrist_model="${wrist_model_left}" tool_changer="${tool_changer_left}" reflect="1" joint_reflect="-1" arm_1_offset="${arm_left_1_joint_offset}" arm_2_offset="${arm_left_2_joint_offset}" arm_3_offset="${arm_left_3_joint_offset}" arm_4_offset="${arm_left_4_joint_offset}" arm_5_offset="${arm_left_5_joint_offset}" arm_6_offset="${arm_left_6_joint_offset}" arm_7_offset="${arm_left_7_joint_offset}" limits_v2="${limits_v2}">
       <origin xyz="$(arg arm_x) $(arg arm_y) $(arg arm_z)" rpy="$(arg arm_roll) $(arg arm_pitch) $(arg arm_yaw)"/>
     </xacro:pal_sea_arm>
@@ -272,5 +275,5 @@
   <xacro:if value="${has_arm_right}">
     <!-- Arm -->
-    <xacro:pal_sea_arm name="arm_right" parent="torso_lift_link" arm_type="${arm_type_right}" wrist_model="${wrist_model_right}" tool_changer="${tool_changer_right}" reflect="1" joint_reflect="1" arm_1_offset="${arm_right_1_joint_offset}" arm_2_offset="${arm_right_2_joint_offset}" arm_3_offset="${arm_right_3_joint_offset}" arm_4_offset="${arm_right_4_joint_offset}" arm_5_offset="${arm_right_5_joint_offset}" arm_6_offset="${arm_right_6_joint_offset}" arm_7_offset="${arm_right_7_joint_offset}">
+    <xacro:pal_sea_arm name="arm_right" parent="torso_lift_link" arm_type="${arm_type_right}" wrist_model="${wrist_model_right}" tool_changer="${tool_changer_right}" reflect="1" joint_reflect="1" arm_1_offset="${arm_right_1_joint_offset}" arm_2_offset="${arm_right_2_joint_offset}" arm_3_offset="${arm_right_3_joint_offset}" arm_4_offset="${arm_right_4_joint_offset}" arm_5_offset="${arm_right_5_joint_offset}" arm_6_offset="${arm_right_6_joint_offset}" arm_7_offset="${arm_right_7_joint_offset}" limits_v2="${limits_v2}">
       <origin xyz="$(arg arm_x) ${-1.0*$(arg arm_y)} $(arg arm_z)" rpy="$(arg arm_roll) ${-1.0*$(arg arm_pitch)} ${-3.14159 -$(arg arm_yaw)}"/>
     </xacro:pal_sea_arm>

Commit message: change name from teleop_basestation to pilot_station

File: tiago_pro_description/robots/tiago_pro.urdf.xacro (robot description, xacro)
@@ -196,7 +196,7 @@
   <!-- Torso -->
   <xacro:include filename="$(find tiago_pro_description)/urdf/torso/torso.urdf.xacro" />
-  <!-- Teleop basestation -->
+  <!-- Teleop pilot station -->
   <xacro:if value="${has_teleop_arms}">
-    <xacro:include filename="$(find tiago_pro_description)/urdf/teleop_basestation/basestation.urdf.xacro" />
+    <xacro:include filename="$(find tiago_pro_description)/urdf/pilot_station/basestation.urdf.xacro" />
   </xacro:if>
   <!-- Calibration constants -->
@@ -214,5 +214,5 @@
   <xacro:if value="${has_teleop_arms}">
     <xacro:if value="${not has_end_effector_teleop_left or not has_end_effector_teleop_right}">
-      <xacro:include filename="$(find tiago_pro_description)/urdf/teleop_basestation/teleop_handle.urdf.xacro" />
+      <xacro:include filename="$(find tiago_pro_description)/urdf/pilot_station/teleop_handle.urdf.xacro" />
     </xacro:if>
     <xacro:if value="${has_end_effector_teleop_left or has_end_effector_teleop_right}">
@@ -238,5 +238,5 @@
   <!-- Teleoperation base station -->
   <xacro:if value="${has_teleop_arms}">
-    <xacro:tiago_pro_teleop_basestation name="teleop_basestation" parent="base_footprint"/>
+    <xacro:tiago_pro_pilot_station name="pilot_station" parent="base_footprint"/>
   </xacro:if>
   <!-- Head -->
@@ -276,8 +276,8 @@
   <!-- Teleop arms FT -->
   <xacro:if value="${has_teleop_arms}">
-    <xacro:pal_sea_arm name="arm_teleop_right" parent="teleop_basestation_base_link" arm_type="${arm_type_teleop_right}" wrist_model="${wrist_model_right}" tool_changer="${tool_changer_teleop_right}" reflect="1" joint_reflect="1" arm_1_offset="${arm_right_1_joint_offset}" arm_2_offset="${arm_right_2_joint_offset}" arm_3_offset="${arm_right_3_joint_offset}" arm_4_offset="${arm_right_4_joint_offset}" arm_5_offset="${arm_right_5_joint_offset}" arm_6_offset="${arm_right_6_joint_offset}" arm_7_offset="${arm_right_7_joint_offset}">
+    <xacro:pal_sea_arm name="arm_teleop_right" parent="pilot_station_base_link" arm_type="${arm_type_teleop_right}" wrist_model="${wrist_model_right}" tool_changer="${tool_changer_teleop_right}" reflect="1" joint_reflect="1" arm_1_offset="${arm_right_1_joint_offset}" arm_2_offset="${arm_right_2_joint_offset}" arm_3_offset="${arm_right_3_joint_offset}" arm_4_offset="${arm_right_4_joint_offset}" arm_5_offset="${arm_right_5_joint_offset}" arm_6_offset="${arm_right_6_joint_offset}" arm_7_offset="${arm_right_7_joint_offset}">
       <origin xyz="0.0 -0.159181203216899 1.21589163274" rpy="-2.06788770984932 0 -1.91986217719377"/>
     </xacro:pal_sea_arm>
-    <xacro:pal_sea_arm name="arm_teleop_left" parent="teleop_basestation_base_link" arm_type="${arm_type_teleop_left}" wrist_model="${wrist_model_left}" tool_changer="${tool_changer_teleop_left}" reflect="1" joint_reflect="-1" arm_1_offset="${arm_left_1_joint_offset}" arm_2_offset="${arm_left_2_joint_offset}" arm_3_offset="${arm_left_3_joint_offset}" arm_4_offset="${arm_left_4_joint_offset}" arm_5_offset="${arm_left_5_joint_offset}" arm_6_offset="${arm_left_6_joint_offset}" arm_7_offset="${arm_left_7_joint_offset}">
+    <xacro:pal_sea_arm name="arm_teleop_left" parent="pilot_station_base_link" arm_type="${arm_type_teleop_left}" wrist_model="${wrist_model_left}" tool_changer="${tool_changer_teleop_left}" reflect="1" joint_reflect="-1" arm_1_offset="${arm_left_1_joint_offset}" arm_2_offset="${arm_left_2_joint_offset}" arm_3_offset="${arm_left_3_joint_offset}" arm_4_offset="${arm_left_4_joint_offset}" arm_5_offset="${arm_left_5_joint_offset}" arm_6_offset="${arm_left_6_joint_offset}" arm_7_offset="${arm_left_7_joint_offset}">
       <origin xyz="0.0 0.159181203216899 1.21589163274" rpy="-2.06788770984932 0 -1.22173047639603"/>
     </xacro:pal_sea_arm>

File: tiago_pro_description/urdf/pilot_station/basestation.urdf.xacro (robot description, xacro)
@@ -13,6 +13,6 @@
 -->
 <robot xmlns:xacro="http://ros.org/wiki/xacro">
-  <xacro:macro name="tiago_pro_teleop_basestation" params="name parent">
-  <!-- Teleoperation base station -->
+  <xacro:macro name="tiago_pro_pilot_station" params="name parent">
+  <!-- Teleop pilot station base link -->
     <link
       name="${name}_base_link">
@@ -36,5 +36,5 @@
           rpy="0 0 0" />
         <geometry>
-            <mesh filename="package://tiago_pro_description/meshes/teleop_basestation/fixed_sit_station.stl" />
+            <mesh filename="package://tiago_pro_description/meshes/pilot_station/fixed_sit_station.stl" />
         </geometry>
         <material
@@ -49,5 +49,5 @@
           rpy="0 0 0" />
         <geometry>
-            <mesh filename="package://tiago_pro_description/meshes/teleop_basestation/fixed_sit_station.stl" />
+            <mesh filename="package://tiago_pro_description/meshes/pilot_station/fixed_sit_station.stl" />
         </geometry>
       </collision>
@@ -66,5 +66,5 @@
         xyz="0 0 0" />
     </joint>
-    <!-- Teleop basestation arm left link -->
+    <!-- Teleop pilot station arm left link -->
     <link name="${name}_arm_left_link"/>
     <joint name="${name}_arm_left_joint" type="fixed">
@@ -74,5 +74,5 @@
       <axis xyz="0 0 0" />
     </joint>
-    <!-- Teleop basestation arm right link -->
+    <!-- Teleop pilot station arm right link -->
     <link name="${name}_arm_right_link"/>
     <joint name="${name}_arm_right_joint" type="fixed">

File: tiago_pro_description/urdf/pilot_station/teleop_handle.urdf.xacro (robot description, xacro)
@@ -36,5 +36,5 @@
         rpy="0 0 0" />
       <geometry>
-          <mesh filename="package://tiago_pro_description/meshes/teleop_basestation/teleop_handle.stl" />
+          <mesh filename="package://tiago_pro_description/meshes/pilot_station/teleop_handle.stl" />
       </geometry>
       <material
@@ -49,5 +49,5 @@
         rpy="0 0 0" />
       <geometry>
-          <mesh filename="package://tiago_pro_description/meshes/teleop_basestation/teleop_handle.stl" />
+          <mesh filename="package://tiago_pro_description/meshes/pilot_station/teleop_handle.stl" />
       </geometry>
     </collision>

Commit message: add enable wrist camera option

File: tiago_pro_description/robots/tiago_pro.urdf.xacro (robot description, xacro)
@@ -26,4 +26,6 @@
   <!-- straight-wrist, spherical-wrist -->
   <xacro:arg name="wrist_model_right" default="spherical-wrist" />
+  <!-- true, false camera on the wrist -->
+  <xacro:arg name="has_wrist_camera" default="False" />
   <!-- False, True -->
   <xacro:arg name="tool_changer_right" default="True" />
@@ -118,4 +120,5 @@
   <xacro:property name="end_effector_teleop_left_name" value="gripper_teleop_left" />
   <xacro:property name="end_effector_teleop_right_name" value="gripper_teleop_right" />
+  <xacro:property name="has_wrist_camera" value="$(arg has_wrist_camera)" />
   <!-- Properties check -->
   <xacro:if value="${arm_type_left not in ['tiago-pro-prototype', 'tiago-pro', 'tiago-pro-s', 'no-arm']}">
@@ -202,4 +205,8 @@
   <!-- Calibration constants -->
   <xacro:include filename="$(arg calibration_offset_dir)/calibration_offset.urdf.xacro" />
+  <!-- Wrist camera -->
+  <xacro:if value="${has_wrist_camera}">
+    <xacro:include filename="$(find pal_sea_arm_description)/urdf/end_effector_camera/end_effector_camera.urdf.xacro" />
+  </xacro:if>
   <!-- Arm -->
   <xacro:if value="${has_arm_right or has_arm_left}">
@@ -209,5 +216,4 @@
   <xacro:if value="${(has_arm_right or has_arm_left) and (has_end_effector_right or has_end_effector_left)}">
     <xacro:include filename="$(find pal_sea_arm_description)/urdf/end_effector/end_effector.urdf.xacro" />
-    <xacro:include filename="$(find pal_sea_arm_description)/urdf/end_effector_camera/end_effector_camera.urdf.xacro" />
   </xacro:if>
   <!-- Trigger Handle for teleop -->
@@ -252,5 +258,7 @@
       <xacro:pal_sea_arm_end_effector name="gripper_left" parent="${end_effector_left_link}" type="${end_effector_left}" tool_changer="${tool_changer_left}" reflect="-1"/>
     </xacro:if>
-    <xacro:pal_sea_arm_end_effector_camera name="gripper_left" parent="${end_effector_left_link}" type="realsense-d435" camera_position="up"/>
+    <xacro:if value="${has_wrist_camera}">
+      <xacro:pal_sea_arm_end_effector_camera name="gripper_left" parent="${end_effector_left_link}" type="realsense-d435" camera_position="up"/>
+    </xacro:if>
     <!-- FT sensors -->
     <xacro:if value="${has_ft_sensor_left}">
@@ -268,5 +276,7 @@
       <xacro:pal_sea_arm_end_effector name="gripper_right" parent="${end_effector_right_link}" type="${end_effector_right}" tool_changer="${tool_changer_right}" reflect="1"/>
     </xacro:if>
-    <xacro:pal_sea_arm_end_effector_camera name="gripper_right" parent="${end_effector_right_link}" type="realsense-d435" camera_position="up"/>
+    <xacro:if value="${has_wrist_camera}">
+      <xacro:pal_sea_arm_end_effector_camera name="gripper_right" parent="${end_effector_right_link}" type="realsense-d435" camera_position="up"/>
+    </xacro:if>
     <!-- FT sensors -->
     <xacro:if value="${has_ft_sensor_right}">

Commit message: Add support for no-wheels

File: tiago_pro_description/robots/tiago_pro.urdf.xacro (robot description, xacro)
@@ -75,4 +75,5 @@
   <xacro:arg name="arm_pitch" default="0.0" />
   <xacro:arg name="arm_yaw" default="-1.2217" />
+  <xacro:arg name="wheel_model" default="moog" />
   <!-- PROPERTIES -->
   <xacro:property name="torque_estimation" value="$(arg torque_estimation)" />
@@ -127,4 +128,5 @@
   <xacro:property name="end_effector_teleop_right_name" value="gripper_teleop_right" />
   <xacro:property name="has_wrist_camera" value="$(arg has_wrist_camera)" />
+  <xacro:property name="wheel_model" value="$(arg wheel_model)" />
   <!-- Properties check -->
   <xacro:if value="${arm_type_left not in ['tiago-pro-prototype', 'tiago-pro', 'tiago-pro-s', 'no-arm']}">
@@ -166,4 +168,7 @@
   <xacro:if value="${laser_model not in ['no-laser', 'sick-571']}">
     <xacro:wrong_laser_model />
+  </xacro:if>
+  <xacro:if value="${wheel_model not in ['moog', 'no-wheels']}">
+    <xacro:wrong_wheel_model />
   </xacro:if>
   <!-- Compatibility check within TC and ft sensors-->

File: tiago_pro_description/ros2_control/ros2_control.urdf.xacro (robot description, xacro)
@@ -112,4 +112,5 @@
     <xacro:arg name="ft_sensor_teleop_left" default="no-ft-sensor"/>
     <xacro:arg name="ft_sensor_teleop_right" default="no-ft-sensor"/>
+    <xacro:arg name="wheel_model" default="moog"/>
     <xacro:arg name="calibration_offset_dir" default="$(find tiago_pro_description)/urdf/calibration" />
     <!-- TODO-->
@@ -127,4 +128,5 @@
     <xacro:property name="has_arm_right" value="${arm_type_right != 'no-arm'}" />
     <xacro:property name="can_device_name" value="can_device" />
+    <xacro:property name="wheel_model" value="$(arg wheel_model)" />
     <xacro:include filename="$(find omni_base_description)/urdf/wheels/wheel.ros2_control.xacro" />
     <xacro:include filename="$(find tiago_pro_description)/urdf/torso/torso.ros2_control.xacro" />
@@ -176,13 +178,15 @@
     <!-- Hardware -->
     <xacro:unless value="$(arg use_sim_time)">
-      <!-- CAN system -->
-      <ros2_control name="ros2_control_tiago_pro_system_can" type="system" rw_rate="100">
-        <hardware>
-          <plugin>robot_control/RobotControl</plugin>
-          <param name="group">can</param>
-        </hardware>
-        <!-- wheels -->
-        <xacro:ros2_control_wheels />
-      </ros2_control>
+      <xacro:if value="${wheel_model == 'moog'}">
+        <!-- CAN system -->
+        <ros2_control name="ros2_control_tiago_pro_system_can" type="system" rw_rate="100">
+          <hardware>
+            <plugin>robot_control/RobotControl</plugin>
+            <param name="group">can</param>
+          </hardware>
+          <!-- wheels -->
+          <xacro:ros2_control_wheels />
+        </ros2_control>
+      </xacro:if>
       <!-- Dynamixels system -->
       <ros2_control name="ros2_control_tiago_pro_system_dynamixel" type="system" rw_rate="100">
@@ -206,4 +210,5 @@
         <!-- arms -->
         <xacro:ros2_control_arms/>
+        <!-- torso -->
         <xacro:ros2_control_torso name="torso_lift" reduction="1.0" />
       </ros2_control>
